File: ch32-examplecluster.kicad_sch (KiCad schematic)
At the start: 19 parts, among them J1 USBC, J2 DEBUG, SW1 RST, SW2 BOOT, U1 CH32V203GxUx, U2 AMS1117-3.3, Y1 X32258MOB4SI 8MHZ

Commit message: finish main mcu and start modules
Connections:
- net CS4: now reaches U1.10 (PA4)
- net CS5: now reaches U1.11 (PA5)
- net CS6: now reaches U1.12 (PA6)
- net CS7: now reaches U1.13 (PA7)
- net SCK: now reaches U1.24 (PB3)
- net MISO: now reaches U1.25 (PB4)
- net MOSI: now reaches U1.26 (PB5)
- net CS0: now reaches U1.6 (PA0)
- net CS1: now reaches U1.7 (PA1)
- net CS2: now reaches U1.8 (PA2)
- net CS3: now reaches U1.9 (PA3)
Other:
- added sheet Module2 (module.kicad_sch)
- added sheet Module3 (module.kicad_sch)
- added sheet Module4 (module.kicad_sch)
- added sheet Module5 (module.kicad_sch)
- added sheet Module6 (module.kicad_sch)
- added sheet Module7 (module.kicad_sch)
- added sheet Module8 (module.kicad_sch)
- moved on the sheet: C3, C4, C5, C6, C7, C8, R3, R4, SW1, SW2, U1, Y1

Commit message: almost finished with schematic
Other:
- sheet Module1 ports: added MISO, MOSI, SCK, SPI_CS; removed none
- sheet Module2 ports: added MISO, MOSI, SCK, SPI_CS; removed none
- sheet Module3 ports: added MISO, MOSI, SCK, SPI_CS; removed none
- sheet Module4 ports: added MISO, MOSI, SCK, SPI_CS; removed none
- sheet Module5 ports: added MISO, MOSI, SCK, SPI_CS; removed none
- sheet Module6 ports: added MISO, MOSI, SCK, SPI_CS; removed none
- sheet Module7 ports: added MISO, MOSI, SCK, SPI_CS; removed none
- sheet Module8 ports: added MISO, MOSI, SCK, SPI_CS; removed none
