File: module.kicad_sch (KiCad schematic)
At the start: 0 parts

Commit message: quickupload
Parts:
- added C9: 100nF, Package_DFN_QFN:QFN-20-1EP_3x3mm_P0.4mm_EP1.65x1.65mm, symbol Device:C_Small
- added TP1: SWIO, symbol Connector:TestPoint
- added U3: CH32V003FxUx, Package_DFN_QFN:QFN-20-1EP_3x3mm_P0.4mm_EP1.65x1.65mm, symbol MCU_WCH_RiscV:CH32V003FxUx
Connections:
- new net +3V3: C9.2, U3.6 (VDD)
- new net GND: C9.1, U3.21 (VSS), U3.4 (VSS)
- new net MISO: U3.14 (PC7)
- new net MOSI: U3.13 (PC6)
- new net SCK: U3.12 (PC5)
- new net SPI_CS: U3.8 (PC1)
- new net SWIO: U3.15 (PD1)

Commit message: almost finished with schematic
Parts:
- added TP17: VDD, symbol Connector:TestPoint
- added TP9: GND, symbol Connector:TestPoint
Connections:
- net +3V3: now also TP17.1
- net GND: now also TP9.1
- net SWIO: now also TP1.1

Commit message: add led
Parts:
- added D1: LED, LED_SMD:LED_Cree-XHP50_3V_HighDensity, symbol Device:LED
- added R5: 330R, symbol Device:R_Small
Connections:
- net +3V3: now also R5.1
- net at U3.11 (PC4): now also D1.1 (K)
- new net: D1.2 (A), R5.2
